File: contr-disp-digitais.kicad_pcb (KiCad board)
At the start: 2 copper layers, 0 parts

Commit message: Revisão de schematics finalizado. Posicionamentos dos componentes do circuito 1 e 2 no PCB editor.
Parts:
- added C1: 2200uF/25V, Capacitor_THT:CP_Radial_D10.0mm_P3.50mm, F.Cu at (94.5, 25.4)
- added C10: 100nF/50V, Capacitor_SMD:C_0805_2012Metric, F.Cu at (89.7, 175.4)
- added C11: 10uF/25V, Capacitor_SMD:CP_Elec_4x5.8, F.Cu at (79.8, 162.1)
- added C12: 10uF/25V, Capacitor_SMD:CP_Elec_4x5.8, F.Cu at (79.8, 167.9)
- added C13: 100nF/50V, Capacitor_SMD:C_0805_2012Metric, F.Cu at (95.3, 167.1)
- added C14: 100nF/50V, Capacitor_SMD:C_0805_2012Metric, F.Cu at (95.3, 171.3)
- added C15: 10uF/25V, Capacitor_SMD:CP_Elec_4x5.8, F.Cu at (79.8, 173.8)
- added C16: 100nF/50V, Capacitor_SMD:C_0805_2012Metric, F.Cu at (95.3, 175.4)
- added C17: 10uF/25V, Capacitor_SMD:CP_Elec_4x5.8, F.Cu at (79.8, 179.6)
- added C18: 100nF/50V, Capacitor_SMD:C_0805_2012Metric, F.Cu at (101.0, 167.1)
- added C19: 100nF/50V, Capacitor_SMD:C_0805_2012Metric, F.Cu at (101.0, 171.3)
- added C2: 2200uF/25V, Capacitor_THT:CP_Radial_D10.0mm_P3.50mm, F.Cu at (94.5, 44.9)
- added C20: 10uF/25V, Capacitor_SMD:CP_Elec_4x5.8, F.Cu at (143.5, 25.5)
- added C21: 100nF/50V, Capacitor_SMD:C_0805_2012Metric, F.Cu at (101.0, 175.4)
- added C22: 10uF/25V, Capacitor_SMD:CP_Elec_4x5.8, F.Cu at (79.8, 185.5)
- added C23: 100nF/50V, Capacitor_SMD:C_0805_2012Metric, F.Cu at (143.5, 29.0)
- added C24: 100nF/50V, Capacitor_SMD:C_0805_2012Metric, F.Cu at (131.0, 47.0)
- added C25: 10uF/25V, Capacitor_SMD:CP_Elec_4x5.8, F.Cu at (130.5, 43.5)
- added C26: 100nF/50V, Capacitor_SMD:C_0805_2012Metric, F.Cu at (153.8, 45.8)
- added C27: 10uF/25V, Capacitor_SMD:CP_Elec_4x5.8, F.Cu at (153.3, 42.2)
- added C28: 100nF/50V, Capacitor_SMD:C_0805_2012Metric, F.Cu at (177.5, 46.0)
- added C29: 10uF/25V, Capacitor_SMD:CP_Elec_4x5.8, F.Cu at (177.0, 42.5)
- added C3: 100nF/50v, Capacitor_THT:C_Disc_D3.4mm_W2.1mm_P2.50mm, F.Cu at (105.0, 25.2)
- added C30: 10uF/25V, Capacitor_SMD:CP_Elec_4x5.8, F.Cu at (167.3, 25.2)
- added C31: 100nF/50V, Capacitor_SMD:C_0805_2012Metric, F.Cu at (167.8, 28.8)
- added C32: 10uF/25V, Capacitor_SMD:CP_Elec_4x5.8, F.Cu at (190.0, 25.0)
- added C33: 100nF/50V, Capacitor_SMD:C_0805_2012Metric, F.Cu at (190.5, 28.5)
- added C4: 100nF/50v, Capacitor_THT:C_Disc_D3.4mm_W2.1mm_P2.50mm, F.Cu at (104.0, 46.2)
- added C5: 100nF/50v, Capacitor_THT:C_Disc_D3.4mm_W2.1mm_P2.50mm, F.Cu at (119.0, 25.0)
- added C6: 100nF/50v, Capacitor_THT:C_Disc_D3.4mm_W2.1mm_P2.50mm, F.Cu at (118.0, 48.5)
- added C7: 100nF/50V, Capacitor_SMD:C_0805_2012Metric, F.Cu at (89.7, 167.1)
- added C8: 10uF/25V, Capacitor_SMD:CP_Elec_4x5.8, F.Cu at (79.8, 156.2)
- added C9: 100nF/50V, Capacitor_SMD:C_0805_2012Metric, F.Cu at (89.7, 171.3)
- added D1: 1N4007, Diode_THT:D_DO-41_SOD81_P10.16mm_Horizontal, F.Cu at (81.0, 25.3)
- added D2: 1N4007, Diode_THT:D_DO-41_SOD81_P10.16mm_Horizontal, F.Cu at (81.0, 38.4)
- added D3: 1N4007, Diode_THT:D_DO-41_SOD81_P10.16mm_Horizontal, F.Cu at (84.5, 25.4)
- added D4: 1N4007, Diode_THT:D_DO-41_SOD81_P10.16mm_Horizontal, F.Cu at (84.5, 38.4)
- added D5: LED, LED_SMD:LED_0805_2012Metric, F.Cu at (121.5, 29.5)
- added D6: LED, LED_SMD:LED_0805_2012Metric, F.Cu at (120.5, 46.6)
- added F1: 0.5A/220V, Fuse:Fuseholder_Clip-5x20mm_Keystone_3512P_Inline_P23.62x7.27mm_D1.02x2.41x1.02x1.57mm_Horizontal, F.Cu at (18.2, 47.3)
- added J1: Conn_01x02, TerminalBlock_Phoenix:TerminalBlock_Phoenix_MKDS-1,5-2-5.08_1x02_P5.08mm_Horizontal, F.Cu at (18.2, 56.7)
- added J2: Conn_01x06, Connector_PinHeader_2.54mm:PinHeader_1x06_P2.54mm_Vertical, F.Cu at (147.5, 16.5)
- added R1: R, Resistor_SMD:R_0805_2012Metric, F.Cu at (85.9, 166.5)
- added R10: R, Resistor_SMD:R_0805_2012Metric, F.Cu at (127.5, 32.0)
- added R11: R, Resistor_SMD:R_0805_2012Metric, F.Cu at (150.9, 35.8)
- added R12: R, Resistor_SMD:R_0805_2012Metric, F.Cu at (150.9, 33.8)
- added R13: R, Resistor_SMD:R_0805_2012Metric, F.Cu at (150.9, 31.8)
- added R14: R, Resistor_SMD:R_0805_2012Metric, F.Cu at (174.6, 36.0)
- added R15: R, Resistor_SMD:R_0805_2012Metric, F.Cu at (174.5, 34.0)
- added R16: R, Resistor_SMD:R_0805_2012Metric, F.Cu at (174.5, 32.0)
- added R17: 1k, Resistor_SMD:R_0805_2012Metric, F.Cu at (121.5, 26.0)
- added R18: 1k, Resistor_SMD:R_0805_2012Metric, F.Cu at (120.5, 50.0)
- added R2: R, Resistor_SMD:R_0805_2012Metric, F.Cu at (85.9, 169.5)
- added R3: R, Resistor_SMD:R_0805_2012Metric, F.Cu at (85.9, 172.4)
- added R4: R, Resistor_SMD:R_0805_2012Metric, F.Cu at (85.9, 175.4)
- added R5: R, Resistor_SMD:R_0805_2012Metric, F.Cu at (85.9, 178.3)
- added R6: R, Resistor_SMD:R_0805_2012Metric, F.Cu at (85.9, 181.3)
- added R7: R, Resistor_SMD:R_0805_2012Metric, F.Cu at (85.9, 184.2)
- added R8: R, Resistor_SMD:R_0805_2012Metric, F.Cu at (127.6, 36.0)
- added R9: R, Resistor_SMD:R_0805_2012Metric, F.Cu at (127.6, 34.0)
- added RV1: Varistor, Varistor:RV_Disc_D12mm_W4.7mm_P7.5mm, F.Cu at (30.0, 54.2)
- added RV2: 10k, Potentiometer_THT:Potentiometer_Bourns_3296W_Vertical, F.Cu at (141.5, 43.0)
- added RV3: 10k, Potentiometer_THT:Potentiometer_Bourns_3296W_Vertical, F.Cu at (137.6, 26.1)
- added RV4: 10k, Potentiometer_THT:Potentiometer_Bourns_3296W_Vertical, F.Cu at (164.5, 42.0)
- added RV5: 10k, Potentiometer_THT:Potentiometer_Bourns_3296W_Vertical, F.Cu at (161.1, 25.5)
- added RV6: 10k, Potentiometer_THT:Potentiometer_Bourns_3296W_Vertical, F.Cu at (188.2, 42.4)
- added RV7: 10k, Potentiometer_THT:Potentiometer_Bourns_3296W_Vertical, F.Cu at (184.1, 26.0)
- added SW1: SW_SPDT, Button_Switch_THT:SW_NKK_BB15AH, F.Cu at (32.5, 42.8)
- added T1: Transformer_1P_2S, Transformer_THT:Transformer_CHK_EI48-8VA_2xSec, F.Cu at (44.2, 50.5)
- added U1: LM7815_TO220, Package_TO_SOT_THT:TO-220-3_Vertical, F.Cu at (109.5, 25.0)
- added U2: LM7915_TO220, Package_TO_SOT_THT:TO-220-3_Vertical, F.Cu at (113.5, 48.5)
- added U3: TL081, Package_DIP:DIP-8_W7.62mm_LongPads, F.Cu at (85.7, 155.4)
- added U4: TL081, Package_DIP:DIP-8_W7.62mm_LongPads, F.Cu at (97.3, 155.4)
- added U5: TL081, Package_DIP:DIP-8_W7.62mm_LongPads, F.Cu at (108.9, 155.4)
- added U6: TL081, Package_DIP:DIP-8_W7.62mm_LongPads, F.Cu at (131.2, 30.8)
- added U7: TL081, Package_DIP:DIP-8_W7.62mm_LongPads, F.Cu at (154.5, 29.9)
- added U8: TL081, Package_DIP:DIP-8_W7.62mm_LongPads, F.Cu at (178.0, 30.4)
Routing:
- net GND: track 0.00 -> 78.5 mm
- net Net-(SW1-B): track 0.00 -> 35.5 mm
- net Net-(J1-Pin_2): track 0.00 -> 32.8 mm
- net Net-(D2-A): track 0.00 -> 31.9 mm
- net Net-(SW1-A): track 0.00 -> 22.1 mm
- net Net-(D1-K): track 0.00 -> 18.2 mm
- net Net-(J1-Pin_1): track 0.00 -> 16.7 mm
- net +15V: track 0.00 -> 6.92 mm
- net Net-(D1-A): track 0.00 -> 2.92 mm
- net Net-(D3-A): track 0.00 -> 2.84 mm
- net -15V: track 0.00 -> 2.50 mm
- net Net-(D5-A): track 0.00 -> 1.65 mm
- net Net-(D6-K): track 0.00 -> 1.59 mm
Other:
- board outline added: 185 x 64 mm
