File: av3/projeto-av3/entradas_analogicas.kicad_sch (KiCad schematic)
At the start: 0 parts

Commit message: Maioria dos esquemáticos finalizados.
Parts:
- added RV1, RV2, RV3, RV4, RV5, RV6, RV7, RV8: 10k, symbol Device:R_Potentiometer
Connections:
- new net +5V: RV1.1, RV2.1, RV3.1, RV4.1, RV5.1, RV6.1, RV7.1, RV8.1
- new net Entrada Analógica 1: RV1.2
- new net Entrada Analógica 2: RV2.2
- new net Entrada Analógica 3: RV3.2
- new net Entrada Analógica 4: RV4.2
- new net Entrada Analógica 5: RV5.2
- new net Entrada Analógica 6: RV6.2
- new net Entrada Analógica 7: RV7.2
- new net Entrada Analógica 8: RV8.2
- new net GND: RV1.3, RV2.3, RV3.3, RV4.3, RV5.3, RV6.3, RV7.3, RV8.3

Commit message: Esquemático finalizado, faltando somente o PCB.
Parts:
- RV1, RV2, RV3, RV4, RV5, RV6, RV7, RV8: footprint (none) -> Potentiometer_THT:Potentiometer_Bourns_3296W_Vertical
Connections:
- net Entrada Analógica 1 renamed ADC0
- net Entrada Analógica 2 renamed ADC1
- net Entrada Analógica 3 renamed ADC2
- net Entrada Analógica 4 renamed ADC3
- net Entrada Analógica 5 renamed ADC4
- net Entrada Analógica 6 renamed ADC5
- net Entrada Analógica 7 renamed ADC6
- net Entrada Analógica 8 renamed ADC7
Changed lines of the file:
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@@
 	(generator_version "8.0")
 	(paper "A4")
-	(global_label "Entrada Analógica 5"
+	(global_label "ADC4"
 		(shape input)
 		(at 54.61 74.93 0)
@@
 		)
 		(property "Intersheetrefs" "${INTERSHEET_REFS}"
-			(at 77.189 74.93 0)
+			(at 62.4333 74.93 0)
 			(effects
 				(font
@@
 		)
 	)
-	(global_label "Entrada Analógica 4"
+	(global_label "ADC3"
 		(shape input)
 		(at 175.26 52.07 0)
@@
 		)
 		(property "Intersheetrefs" "${INTERSHEET_REFS}"
-			(at 197.839 52.07 0)
+			(at 183.0833 52.07 0)
 			(effects
 				(font
@@
 		)
 	)
-	(global_label "Entrada Analógica 7"
+	(global_label "ADC6"
 		(shape input)
 		(at 135.89 74.93 0)
@@
 		)
 		(property "Intersheetrefs" "${INTERSHEET_REFS}"
-			(at 158.469 74.93 0)
+			(at 143.7133 74.93 0)
 			(effects
 				(font
@@
 		)
 	)
-	(global_label "Entrada Analógica 1"
+	(global_label "ADC0"
 		(shape input)
 		(at 54.61 52.07 0)
@@
 		)
 		(property "Intersheetrefs" "${INTERSHEET_REFS}"
-			(at 77.189 52.07 0)
+			(at 62.4333 52.07 0)
 			(effects
 				(font
@@
 		)
 	)
-	(global_label "Entrada Analógica 6"
+	(global_label "ADC5"
 		(shape input)
 		(at 95.25 74.93 0)
@@
 		)
 		(property "Intersheetrefs" "${INTERSHEET_REFS}"
-			(at 117.829 74.93 0)
+			(at 103.0733 74.93 0)
 			(effects
 				(font
@@
 		)
 	)
-	(global_label "Entrada Analógica 2"
+	(global_label "ADC1"
 		(shape input)
 		(at 95.25 52.07 0)
@@
 		)
 		(property "Intersheetrefs" "${INTERSHEET_REFS}"
-			(at 117.829 52.07 0)
+			(at 103.0733 52.07 0)
 			(effects
 				(font
@@
 		)
 	)
-	(global_label "Entrada Analógica 8"
+	(global_label "ADC7"
 		(shape input)
 		(at 175.26 74.93 0)
@@
 		)
 		(property "Intersheetrefs" "${INTERSHEET_REFS}"
-			(at 197.839 74.93 0)
+			(at 183.0833 74.93 0)
 			(effects
 				(font
@@
 		)
 	)
-	(global_label "Entrada Analógica 3"
+	(global_label "ADC2"
 		(shape input)
 		(at 135.89 52.07 0)
@@
 		)
 		(property "Intersheetrefs" "${INTERSHEET_REFS}"
-			(at 158.469 52.07 0)
+			(at 143.7133 52.07 0)
 			(effects
 				(font
@@
 			)
 		)
-		(property "Footprint" ""
+		(property "Footprint" "Potentiometer_THT:Potentiometer_Bourns_3296W_Vertical"
 			(at 171.45 52.07 0)
 			(effects
@@
 			)
 		)
-		(property "Footprint" ""
+		(property "Footprint" "Potentiometer_THT:Potentiometer_Bourns_3296W_Vertical"
 			(at 91.44 74.93 0)
 			(effects
@@
 			)
 		)
-		(property "Footprint" ""
+		(property "Footprint" "Potentiometer_THT:Potentiometer_Bourns_3296W_Vertical"
 			(at 132.08 74.93 0)
 			(effects
@@
 			)
 		)
-		(property "Footprint" ""
+		(property "Footprint" "Potentiometer_THT:Potentiometer_Bourns_3296W_Vertical"
 			(at 50.8 52.07 0)
 			(effects
@@
 			)
 		)
-		(property "Footprint" ""
+		(property "Footprint" "Potentiometer_THT:Potentiometer_Bourns_3296W_Vertical"
 			(at 50.8 74.93 0)
 			(effects
@@
 			)
 		)
-		(property "Footprint" ""
+		(property "Footprint" "Potentiometer_THT:Potentiometer_Bourns_3296W_Vertical"
 			(at 132.08 52.07 0)
 			(effects
@@
 			)
 		)
-		(property "Footprint" ""
+		(property "Footprint" "Potentiometer_THT:Potentiometer_Bourns_3296W_Vertical"
 			(at 91.44 52.07 0)
 			(effects
@@
 			)
 		)
-		(property "Footprint" ""
+		(property "Footprint" "Potentiometer_THT:Potentiometer_Bourns_3296W_Vertical"
 			(at 171.45 74.93 0)
 			(effects
