File: av3/projeto-av3/lcd16x02.kicad_sch (KiCad schematic)
At the start: 1 part

Commit message: Esquemático finalizado, faltando somente o PCB.
Parts:
- removed DS1: WC1602A, Display:WC1602A, symbol Display_Character:WC1602A
- added DS1: HY1602E, Display:HY1602E, symbol Display_Character:HY1602E
- added RV9: 10K, Potentiometer_THT:Potentiometer_Bourns_3296W_Vertical, symbol Device:R_Potentiometer
Connections:
- net D4: now also DS1.13 (DB4)
- net D5: now also DS1.14 (DB5)
- net D6: now also DS1.15 (DB6)
- net D7: now also DS1.16 (DB7)
- net GND: now also DS1.1 (LEDK), DS1.10 (DB1), DS1.11 (DB2), DS1.12 (DB3), DS1.3 (VSS), DS1.7 (R/~{W}), DS1.9 (DB0), RV9.1
- new net: DS1.5 (Vo), RV9.2
- new net +5V: DS1.2 (LEDA), DS1.4 (VDD), RV9.3
- new net E: DS1.8 (E)
- new net RS: DS1.6 (RS)
