File: av3/projeto-av3/saidas_digitais_rele.kicad_sch3.kicad_sch (KiCad schematic)
At the start: 40 parts, among them J10 Conn_01x03, J11 Conn_01x03, J12 Conn_01x03, J13 Conn_01x03, J14 Conn_01x03, J15 Conn_01x03, J16 Conn_01x03, J9 Conn_01x03, K1 SANYOU_SRD_Form_C, K2 SANYOU_SRD_Form_C, K3 SANYOU_SRD_Form_C, K4 SANYOU_SRD_Form_C, K5 SANYOU_SRD_Form_C, K6 SANYOU_SRD_Form_C, K7 SANYOU_SRD_Form_C, K8 SANYOU_SRD_Form_C, Q1 BC548, Q2 BC548, Q3 BC548, Q4 BC548, Q5 BC548, Q6 BC548, Q7 BC548, Q8 BC548

Commit message: Maioria das conexões do PBC feitas, e erros faltando corrigir.
Connections:
- net +5V: now also K1.2; no longer K1.3
- net at D17.2 (A), Q1.1 (C): now also K1.5; no longer K1.1
- net at K1.4: now also J9.3 (Pin_3)
- net at J9.2 (Pin_2): now also K1.1; no longer K1.5
- net at J9.1 (Pin_1): now also K1.3
Changed lines of the file:
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@@
+	)
+	(junction
+		(at 57.15 38.1)
+		(diameter 0)
+		(color 0 0 0 0)
 	)
 	(junction
@@
 	)
 	(junction
+		(at 57.15 22.86)
+		(diameter 0)
+		(color 0 0 0 0)
+	)
+	(junction
 		(at 226.06 83.82)
 		(diameter 0)
@@
 	)
 	(junction
-		(at 57.15 38.1)
-		(diameter 0)
-		(color 0 0 0 0)
-	)
-	(junction
 		(at 130.81 80.01)
 		(diameter 0)
 		(color 0 0 0 0)
 	)
-	(junction
-		(at 54.61 22.86)
-		(diameter 0)
-		(color 0 0 0 0)
-	)
 	(wire
 		(pts
@@
 	(wire
 		(pts
-			(xy 54.61 22.86) (xy 57.15 22.86)
-		)
-		(stroke
-			(width 0)
-			(type default)
-		)
-	)
-	(wire
-		(pts
 			(xy 149.86 96.52) (xy 138.43 96.52)
 		)
@@
 	(wire
 		(pts
+			(xy 69.85 38.1) (xy 74.93 38.1)
+		)
+		(stroke
+			(width 0)
+			(type default)
+		)
+	)
+	(wire
+		(pts
 			(xy 163.83 135.89) (xy 163.83 149.86)
 		)
@@
 	(wire
 		(pts
-			(xy 69.85 38.1) (xy 74.93 38.1)
-		)
-		(stroke
-			(width 0)
-			(type default)
-		)
-	)
-	(wire
-		(pts
 			(xy 236.22 83.82) (xy 242.57 83.82)
 		)
@@
 	(wire
 		(pts
-			(xy 48.26 22.86) (xy 54.61 22.86)
+			(xy 48.26 22.86) (xy 57.15 22.86)
 		)
 		(stroke
@@
 		(lib_id "Relay:SANYOU_SRD_Form_C")
 		(at 62.23 30.48 0)
-		(mirror y)
+		(mirror x)
 		(unit 1)
 		(exclude_from_sim no)
@@
 		(dnp no)
 		(property "Reference" "K1"
-			(at 76.454 29.972 0)
+			(at 48.006 30.988 0)
 			(effects
 				(font
@@
 		)
 		(property "Value" "SANYOU_SRD_Form_C"
-			(at 93.98 27.686 0)
+			(at 30.48 33.274 0)
 			(effects
 				(font
@@
 		)
 		(property "Footprint" "Relay_THT:Relay_SPDT_SANYOU_SRD_Series_Form_C"
-			(at 50.8 31.75 0)
-			(effects
-				(font
+			(at 73.66 29.21 0)
+			(effects
+				(font
