File: av3/projeto-av3/av3.kicad_pcb (KiCad board)
At the start: 2 copper layers, 146 parts, among them J1 Conn_01x02, J10 Jack-DC, J11 Conn_01x03, J12 Conn_01x03, J13 Conn_01x03, J14 Conn_01x03, J15 Conn_01x03, J16 Conn_01x03, J17 Conn_01x03, J18 Conn_02x03_Odd_Even, J19 Conn_01x02, J2 Conn_01x02, J3 Conn_01x02, J4 Conn_01x02, J5 Conn_01x03, J6 DE9_Plug, J7 Conn_01x02, J8 Conn_01x02, J9 Conn_01x02, K1 SANYOU_SRD_Form_C, K2 SANYOU_SRD_Form_C, K3 SANYOU_SRD_Form_C, K4 SANYOU_SRD_Form_C, K5 SANYOU_SRD_Form_C, K6 SANYOU_SRD_Form_C, K7 SANYOU_SRD_Form_C, K8 SANYOU_SRD_Form_C, Q1 BC548, Q2 BC548, Q3 BC548, Q4 BC548, Q5 BC548, Q6 BC548, Q7 BC548, Q8 BC548, SW1 SW_Push, SW10 SW_Push, SW11 SW_Push, SW12 SW_Push, SW13 SW_Push, SW14 SW_Push, SW15 SW_Push, SW16 SW_Push, SW17 SW_Push, SW2 SW_Push, SW3 SW_Push, SW4 SW_Push, SW5 SW_Push, SW6 SW_Push, SW7 SW_Push, SW8 SW_Push, SW9 SW_Push, U1 4N25, U10 4N25, U11 L7805, U2 4N25, U3 4N25, U4 4N25, U5 ATmega2560-16A, U6 MAX232, U7 4N25, U8 4N25, U9 4N25, Y1 16MHz

Commit message: Referencias de componentes resetados; Progresso de 20% no PCB;
Parts:
- moved J9 212.8 mm to (-4.80, 288.0)
- moved D17 196.7 mm to (-6.26, 257.6)
- moved J10 195.8 mm to (12.8, 288.2)
- moved C10 187.7 mm to (202.1, 243.4), turned to -90 degrees
- moved D18 186.7 mm to (10.4, 258.6)
- moved Y1 186.3 mm to (198.0, 238.5)
- moved C3 185.2 mm to (176.3, 354.3)
- moved C2 185.2 mm to (192.2, 339.0)
- moved C4 185.2 mm to (176.3, 339.7)
- moved C6 185.2 mm to (176.3, 349.4)
- moved J17 185.2 mm to (195.5, 254.3)
- moved J18 185.2 mm to (194.9, 321.9)
- moved SW17 185.2 mm to (205.9, 251.4)
- moved U10 185.2 mm to (184.5, 343.2)
- moved U9 185.2 mm to (198.2, 223.3)
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- renumbered C7 to C1, C1 to C10, C2 to C11, C9 to C2, C6 to C3, C3 to C4, C4 to C5, C5 to C6, C10 to C7, C11 to C8, C12 to C9, D13 to D10, D10 to D11, D15 to D12, D17 to D13, D12 to D14, D14 to D15, D9 to D17, D4 to D2, D6 to D3, D8 to D4, D2 to D5, D3 to D6, D5 to D7, D7 to D8, D11 to D9, J11 to J10, J12 to J11, J13 to J12, J14 to J13, J15 to J14, J16 to J15, J17 to J16, J18 to J17, J6 to J18, J10 to J19, J19 to J2, J4 to J3, J8 to J4, J2 to J5, J3 to J6, J9 to J8, J5 to J9, R4 to R10, R7 to R11, R10 to R12, R19 to R13, R20 to R14, R22 to R15, R18 to R16, R25 to R17, R23 to R18, R28 to R19, R5 to R2, R26 to R20, R29 to R22, R24 to R23, R27 to R24, R14 to R25, R15 to R26, R16 to R27, R17 to R28, R13 to R29, R8 to R3, R11 to R4, R3 to R5, R9 to R7, R12 to R8, R2 to R9, U6 to U10, U7 to U5, U8 to U6, U9 to U7, U10 to U8, U5 to U9
Routing:
- net +5V: track 0.00 -> 146.3 mm
- net Net-(U11-IN): track 0.00 -> 29.1 mm
- net Net-(D5-K): track 0.00 -> 16.7 mm
- net Net-(D8-K): track 0.00 -> 16.7 mm
- net Net-(D7-K): track 0.00 -> 16.7 mm
- net Net-(D6-K): track 0.00 -> 16.5 mm
- net Net-(D14-K): track 0.00 -> 16.5 mm
- net Net-(D16-K): track 0.00 -> 16.5 mm
- net Net-(D15-K): track 0.00 -> 16.5 mm
- net Net-(D11-K): track 0.00 -> 16.5 mm
- net Net-(J1-Pin_1): track 0.00 -> 9.50 mm
- net Net-(J2-Pin_1): track 0.00 -> 9.47 mm
- net Net-(J4-Pin_1): track 0.00 -> 9.45 mm
- net Net-(J3-Pin_1): track 0.00 -> 9.45 mm
- net Net-(J8-Pin_1): track 0.00 -> 9.26 mm
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Other:
- board outline added: 272 x 185 mm

Commit message: Maioria das conexões do PBC feitas, e erros faltando corrigir.
Parts:
- moved C6 285.9 mm to (161.2, 63.9)
- moved C1 280.7 mm to (151.8, 73.7), turned to 90 degrees
- moved C3 277.0 mm to (168.2, 77.4), turned to 90 degrees
- moved U10 272.6 mm to (162.0, 71.6), turned to 180 degrees
- moved C4 268.4 mm to (168.2, 71.4), turned to 90 degrees
- moved C2 267.0 mm to (156.2, 74.4), turned to 90 degrees
- moved C5 266.1 mm to (161.8, 78.9), turned to 180 degrees
- moved J18 254.0 mm to (186.7, 68.1), turned to 90 degrees
- moved J17 179.8 mm to (90.3, 108.5)
- moved SW17 178.9 mm to (100.8, 106.8)
- moved R37 178.9 mm to (101.7, 114.9)
- moved U9 146.6 mm to (122.0, 98.0)
- moved C11 145.4 mm to (117.5, 119.5)
- moved Y1 145.4 mm to (122.0, 114.5)
- moved C10 145.2 mm to (126.5, 119.5)
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Routing:
- net +5V: track 146.3 -> 486.6 mm, vias 0 -> 4
- net L1: track 0.00 -> 105.8 mm, vias 0 -> 10
- net D7: track 0.00 -> 92.3 mm, vias 0 -> 2
- net Net-(DS1-Vo): track 0.00 -> 90.8 mm
- net D6: track 0.00 -> 90.5 mm, vias 0 -> 2
- net D5: track 0.00 -> 88.9 mm, vias 0 -> 2
- net I.7: track 7.14 -> 96.0 mm
- net E: track 0.00 -> 88.0 mm, vias 0 -> 2
- net D4: track 0.00 -> 87.3 mm, vias 0 -> 2
- net RS: track 0.00 -> 87.0 mm, vias 0 -> 2
- net L2: track 0.00 -> 86.5 mm, vias 0 -> 10
- net C2: track 0.00 -> 84.5 mm
- net L3: track 0.00 -> 83.9 mm, vias 0 -> 8
- net O.7: track 0.00 -> 83.8 mm, vias 0 -> 1
- net C1: track 0.00 -> 83.0 mm, vias 0 -> 1
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- added copper zone on B.Cu, net GND
- added copper zone on F.Cu, net GND
Other:
- board size 272 x 185 mm -> 189.5 x 178 mm

Commit message: Montagem base finalizada.
Routing:
- net +5V: track 486.6 -> 702.1 mm, vias 4 -> 5
- net Net-(U9-VCC-Pad10): track 0.00 -> 32.2 mm, vias 0 -> 3
- net Net-(D22-A): track 0.00 -> 10.9 mm
- net Net-(D19-A): track 0.00 -> 10.7 mm
- net Net-(D20-A): track 0.00 -> 10.7 mm
- net Net-(D17-A): track 0.00 -> 10.6 mm
- net Net-(D18-A): track 0.00 -> 10.5 mm
- net Net-(D21-A): track 0.00 -> 9.57 mm
- net Net-(D23-A): track 0.00 -> 9.31 mm
- net Net-(D24-A): track 0.00 -> 9.30 mm
- net L2: track 86.5 -> 93.0 mm
- net Net-(Q5-B): track 0.00 -> 4.21 mm
- net Net-(Q3-B): track 0.00 -> 4.18 mm
- net Net-(Q8-B): track 0.00 -> 4.18 mm
- net Net-(Q7-B): track 0.00 -> 4.18 mm
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